File: kicad/biju_saturn_lamp.kicad_sch (KiCad schematic)
At the start: 24 parts, among them J1 Barrel_Jack, J2 Conn_01x06, J3 Conn_01x02, J4 Conn_01x02, J5 Conn_01x02, SW1 SW_Push, U1 Pico, U2 74HC595, U3 PAM8302AAD

Commit message: update pcb
Connections:
- net GND: now also U1.18 (GND), U1.23 (GND)
Changed lines of the file:
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@@
+    )
+  )
+  (symbol (lib_id "power:GND") (at 26.416 88.392 270) (unit 1)
+    (in_bom yes) (on_board yes) (dnp no) (fields_autoplaced)
+    (property "Reference" "#PWR015" (at 20.066 88.392 0)
+      (effects (font (size 1.27 1.27)) hide)
+    )
+    (property "Value" "GND" (at 22.86 88.392 90)
+      (effects (font (size 1.27 1.27)) (justify right))
+    )
+    (property "Footprint" "" (at 26.416 88.392 0)
+      (effects (font (size 1.27 1.27)) hide)
+    )
+    (property "Datasheet" "" (at 26.416 88.392 0)
+      (effects (font (size 1.27 1.27)) hide)
+    )
+    (pin "1")
+    (instances
+      (project "biju_saturn_lamp"
+        (path "/ad563cc9-592a-4a72-b118-713be0da33dd"
+          (reference "#PWR015") (unit 1)
+        )
+      )
     )
   )
@@
         )
       )
+    )
+  )
+  (symbol (lib_id "power:GND") (at 61.976 88.392 90) (unit 1)
+    (in_bom yes) (on_board yes) (dnp no) (fields_autoplaced)
+    (property "Reference" "#PWR014" (at 68.326 88.392 0)
+      (effects (font (size 1.27 1.27)) hide)
+    )
+    (property "Value" "GND" (at 65.532 88.392 90)
+      (effects (font (size 1.27 1.27)) (justify right))
+    )
+    (property "Footprint" "" (at 61.976 88.392 0)
+      (effects (font (size 1.27 1.27)) hide)
+    )
+    (property "Datasheet" "" (at 61.976 88.392 0)
+      (effects (font (size 1.27 1.27)) hide)
+    )
+    (pin "1")
+    (instances
+      (project "biju_saturn_lamp"
+        (path "/ad563cc9-592a-4a72-b118-713be0da33dd"
+          (reference "#PWR014") (unit 1)
+        )
+      )

Commit message: fix on-off switch
Connections:
- net 3v3_EN: no longer J5.1 (Pin_1)
- net GND: no longer J5.2 (Pin_2), SW1.2
- net VCC: now also J5.1 (Pin_1), SW1.2; no longer J1.1
- new net: J1.1, J5.2 (Pin_2)
Other:
- moved on the sheet: J5
Changed lines of the file:
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@@
+    (stroke (width 0) (type default))
+  )
+  (wire (pts (xy 39.624 25.146) (xy 39.624 25.908))
     (stroke (width 0) (type default))
   )
@@
     (stroke (width 0) (type default))
   )
+  (wire (pts (xy 39.624 25.908) (xy 40.894 25.908))
+    (stroke (width 0) (type default))
+  )
+  (wire (pts (xy 37.084 26.162) (xy 36.576 26.162))
+    (stroke (width 0) (type default))
+  )
   (wire (pts (xy 116.586 132.588) (xy 124.968 132.588))
     (stroke (width 0) (type default))
   )
   (wire (pts (xy 103.632 132.588) (xy 108.966 132.588))
+    (stroke (width 0) (type default))
+  )
+  (wire (pts (xy 37.084 25.146) (xy 37.084 26.162))
     (stroke (width 0) (type default))
   )
@@
     )
   )
+  (global_label "VCC" (shape input) (at 94.742 98.044 0) (fields_autoplaced)
+    (effects (font (size 1.27 1.27)) (justify left))
+    (property "Intersheetrefs" "${INTERSHEET_REFS}" (at 101.3558 98.044 0)
+      (effects (font (size 1.27 1.27)) (justify left) hide)
+    )
+  )
   (global_label "VCC" (shape input) (at 79.756 52.832 180) (fields_autoplaced)
     (effects (font (size 1.27 1.27)) (justify right))
@@
     )
   )
-  (global_label "VCC" (shape input) (at 36.576 26.162 0) (fields_autoplaced)
+  (global_label "VCC" (shape input) (at 40.894 25.908 0) (fields_autoplaced)
     (effects (font (size 1.27 1.27)) (justify left))
-    (property "Intersheetrefs" "${INTERSHEET_REFS}" (at 43.1104 26.162 0)
+    (property "Intersheetrefs" "${INTERSHEET_REFS}" (at 47.4284 25.908 0)
       (effects (font (size 1.27 1.27)) (justify left) hide)
     )
@@
         (path "/ad563cc9-592a-4a72-b118-713be0da33dd"
           (reference "#PWR014") (unit 1)
-        )
-      )
-    )
-  )
-  (symbol (lib_id "power:GND") (at 94.742 98.044 90) (unit 1)
-    (in_bom yes) (on_board yes) (dnp no) (fields_autoplaced)
-    (property "Reference" "#PWR09" (at 101.092 98.044 0)
-      (effects (font (size 1.27 1.27)) hide)
-    )
-    (property "Value" "GND" (at 98.806 98.679 90)
-      (effects (font (size 1.27 1.27)) (justify right))
-    )
-    (property "Footprint" "" (at 94.742 98.044 0)
-      (effects (font (size 1.27 1.27)) hide)
-    )
-    (property "Datasheet" "" (at 94.742 98.044 0)
-      (effects (font (size 1.27 1.27)) hide)
-    )
-    (pin "1")
-    (instances
-      (project "biju_saturn_lamp"
-        (path "/ad563cc9-592a-4a72-b118-713be0da33dd"
-          (reference "#PWR09") (unit 1)
         )
       )
@@
     )
   )
-  (symbol (lib_id "Connector_Generic:Conn_01x02") (at 132.842 97.028 0) (unit 1)
+  (symbol (lib_id "Connector_Generic:Conn_01x02") (at 39.624 20.066 270) (mirror x) (unit 1)
     (in_bom yes) (on_board yes) (dnp no)
-    (property "Reference" "J5" (at 125.73 91.694 0)
-      (effects (font (size 1.27 1.27)) (justify left))
-    )
-    (property "Value" "Conn_01x02" (at 125.73 94.234 0)
-      (effects (font (size 1.27 1.27)) (justify left))
-    )
-    (property "Footprint" "TerminalBlock_Phoenix:TerminalBlock_Phoenix_MKDS-1,5-2_1x02_P5.00mm_Horizontal" (at 132.842 97.028 0)
-      (effects (font (size 1.27 1.27)) hide)
-    )
-    (property "Datasheet" "~" (at 132.842 97.028 0)
-      (effects (font (size 1.27 1.27)) hide)
-    )
+    (property "Reference" "J5" (at 44.958 27.178 0)
+      (effects (font (size 1.27 1.27)) (justify left))
+    )
+    (property "Value" "Conn_01x02" (at 42.418 27.178 0)
+      (effects (font (size 1.27 1.27)) (justify left))
+    )
+    (property "Footprint" "TerminalBlock_Phoenix:TerminalBlock_Phoenix_MKDS-1,5-2_1x02_P5.00mm_Horizontal" (at 39.624 20.066 0)
+      (effects (font (size 1.27 1.27)) hide)
+    )
+    (property "Datasheet" "~" (at 39.624 20.066 0)
+      (effects (font (size 1.27 1.27)) hide)
+    )
